File: hardware/DIYduino.kicad_pcb (KiCad board)
At the start: 2 copper layers, 68.6 x 53.3 mm, 37 parts, among them P1 Power, P2 Analog, P3 Digital, P4 Digital, P5 CONN_1, P6 CONN_1, P7 CONN_1, P8 CONN_1, SW1 SW_RESET, U1 ATmega32U4-AU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

Commit message: update
Parts:
- removed the G*** at (164.2, 107.4)
- added G***: LOGO, DIYduino:szdiy_logo, B.Cu at (163.0, 104.4)
Other:
- board text added: "https://github.com/szdiy/DIYduino"
- board text added: "v1.0"
- board text removed: "https://github.com/danfei/DIYduino"
- board text removed: "v0.2"

Commit message: update
Connections:
- C6 pad 2: +5C -> Net-(C6-Pad2)
- U1 pad 6: +5C -> Net-(C6-Pad2)
Routing:
- net Net-(C6-Pad2): track 0.00 -> 13.6 mm, vias 0 -> 2
- net +5C: track 200.6 -> 190.5 mm
Changed lines of the file:
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@@
 (kicad_pcb (version 4) (host pcbnew 4.0.5+dfsg1-4)
   (general
-    (links 95)
+    (links 94)
     (no_connects 0)
-    (area 104.572999 71.542 180.166572 127.694)
+    (area 110.922999 72.949999 179.653001 126.440001)
     (thickness 1.6)
     (drawings 81)
-    (tracks 536)
+    (tracks 538)
     (zones 0)
     (modules 37)
-    (nets 48)
+    (nets 49)
   )
   (page A4)
@@
     (34 B.Paste user)
     (35 F.Paste user)
-    (36 B.SilkS user)
-    (37 F.SilkS user)
+    (36 B.SilkS user hide)
+    (37 F.SilkS user hide)
     (38 B.Mask user)
     (39 F.Mask user)
@@
   (net 46 "Net-(D1-Pad1)")
   (net 47 "Net-(D2-Pad1)")
+  (net 48 "Net-(C6-Pad2)")
   (net_class Default "This is the default net class."
     (clearance 0.2)
@@
     (add_net "Net-(C1-Pad1)")
     (add_net "Net-(C2-Pad1)")
+    (add_net "Net-(C6-Pad2)")
     (add_net "Net-(CONN1-Pad2)")
     (add_net "Net-(CONN1-Pad3)")
@@
       (net 1 GND))
     (pad 2 thru_hole circle (at 5 0) (size 1.3 1.3) (drill 0.8) (layers *.Cu *.Mask F.SilkS)
-      (net 15 +5C))
+      (net 48 "Net-(C6-Pad2)"))
     (model Capacitors_ThroughHole.3dshapes/C_Rect_L7_W2_P5.wrl
       (at (xyz 0.098425 0 0))
@@
       (net 1 GND))
     (pad 6 smd rect (at -5.7 0 180) (size 1.5 0.55) (layers F.Cu F.Paste F.Mask)
-      (net 15 +5C))
+      (net 48 "Net-(C6-Pad2)"))
     (pad 7 smd rect (at -5.7 0.8 180) (size 1.5 0.55) (layers F.Cu F.Paste F.Mask)
       (net 15 +5C))
@@
   (segment (start 168.9639 94.265) (end 168.9639 90.3312) (width 0.4) (layer B.Cu) (net 14))
   (segment (start 168.698 89.015) (end 168.698 90.0653) (width 0.4) (layer B.Cu) (net 14))
+  (segment (start 169.598 110.565) (end 168.573 111.59) (width 0.55) (layer F.Cu) (net 15))
+  (segment (start 168.573 111.59) (end 166.498 111.59) (width 0.55) (layer F.Cu) (net 15))
+  (segment (start 169.598 109.19) (end 169.598 110.565) (width 0.55) (layer F.Cu) (net 15))
+  (segment (start 168.198 109.09) (end 169.498 109.09) (width 0.55) (layer F.Cu) (net 15))
+  (segment (start 169.498 109.09) (end 169.598 109.19) (width 0.55) (layer F.Cu) (net 15))
   (segment (start 164.898 100.19) (end 164.898 98.885092) (width 0.55) (layer F.Cu) (net 15))
   (segment (start 164.898 98.885092) (end 166.684591 97.098501) (width 0.55) (layer F.Cu) (net 15))
@@
   (segment (start 176.094499 97.098501) (end 176.569501 96.623499) (width 0.55) (layer F.Cu) (net 15))
   (segment (start 176.569501 96.623499) (end 177.268 95.925) (width 0.55) (layer F.Cu) (net 15))
-  (segment (start 166.498 111.59) (end 166.498 114.34) (width 0.55) (layer F.Cu) (net 15))
-  (segment (start 166.498 114.34) (end 168.448 116.29) (width 0.55) (layer F.Cu) (net 15))
-  (segment (start 168.198 109.09) (end 169.278002 109.09) (width 0.55) (layer F.Cu) (net 15))
-  (segment (start 169.278002 109.09) (end 169.423001 109.234999) (width 0.55) (layer F.Cu) (net 15))
-  (segment (start 169.423001 109.234999) (end 169.423001 115.314999) (width 0.55) (layer F.Cu) (net 15))
-  (segment (start 169.423001 115.314999) (end 169.097999 115.640001) (width 0.55) (layer F.Cu) (net 15))
-  (segment (start 169.097999 115.640001) (end 168.448 116.29) (width 0.55) (layer F.Cu) (net 15))
   (segment (start 168.198 109.09) (end 167.117998 109.09) (width 0.55) (layer F.Cu) (net 15))
   (segment (start 167.117998 109.09) (end 166.814898 108.7869) (width 0.55) (layer F.Cu) (net 15))
   (segment (start 166.814898 108.7869) (end 166.814898 105.09) (width 0.55) (layer F.Cu) (net 15))
-  (segment (start 168.198 105.89) (end 166.898 105.89) (width 0.55) (layer F.Cu) (net 15))
-  (segment (start 166.898 105.89) (end 166.814898 105.806898) (width 0.55) (layer F.Cu) (net 15))
-  (segment (start 166.814898 105.806898) (end 166.814898 105.09) (width 0.55) (layer F.Cu) (net 15))
   (segment (start 164.898 101.49) (end 164.898 101.065) (width 0.55) (layer F.Cu) (net 15))
   (segment (start 164.898 101.065) (end 164.898 100.19) (width 0.55) (layer F.Cu) (net 15))
@@
   (segment (start 139.748 101.99) (end 135.2851 106.4529) (width 0.4) (layer B.Cu) (net 47))
   (segment (start 116 106) (end 117.3503 106) (width 0.4) (layer B.Cu) (net 47))
+  (segment (start 170.561 108.99) (end 170.561 114.177) (width 0.55) (layer F.Cu) (net 48))
+  (segment (start 170.561 114.177) (end 168.448 116.29) (width 0.55) (layer F.Cu) (net 48))
+  (segment (start 170.561 105.918) (end 170.561 108.99) (width 0.55) (layer B.Cu) (net 48))
+  (via (at 170.561 108.99) (size 0.6) (drill 0.4) (layers F.Cu B.Cu) (net 48))
+  (segment (start 168.198 105.89) (end 170.533 105.89) (width 0.55) (layer F.Cu) (net 48))
+  (segment (start 170.533 105.89) (end 170.561 105.918) (width 0.55) (layer F.Cu) (net 48))
+  (via (at 170.561 105.918) (size 0.6) (drill 0.4) (layers F.Cu B.Cu) (net 48))
   (zone (net 1) (net_name GND) (layer F.Cu) (hatch edge 0.508)
     (connect_pads (clearance 0.508))
