File: hardware/DIYduino.sch (KiCad schematic (older format))
At the start: 35 parts, among them P1 Power, P2 Analog, P3 Digital, P4 Digital, P5 CONN_1, P6 CONN_1, P7 CONN_1, P8 CONN_1, SW1 SW_RESET, U1 ATmega32U4-AU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

Commit message: update
Parts:
- CONN1: symbol USB_B -> USB_B-RESCUE-DIYduino
- U1: symbol ATmega32U4-AU -> ATmega32U4-AU-RESCUE-DIYduino
- renumbered R7 to R6, R6 to R7
Changed lines of the file:
@@
 EESchema Schematic File Version 2
+LIBS:DIYduino-rescue
 LIBS:power
 LIBS:device
@@
 LIBS:valves
 LIBS:LCD7th
-LIBS:reduino-cache
+LIBS:DIYduino-cache
 EELAYER 25 0
 EELAYER END
@@
 Shield for Arduino that uses\nthe same pin disposition\nlike "Uno" board Rev 3.
 $Comp
-L ATmega32U4-AU U1
+L ATmega32U4-AU-RESCUE-DIYduino U1
 U 1 1 572024B2
 P 3800 2850
@@
 TX_LED
 $Comp
-L R_Small R7
+L R_Small R6
 U 1 1 57205DB6
 P 6950 4600
-F 0 "R7" H 6980 4620 50  0000 L CNN
+F 0 "R6" H 6980 4620 50  0000 L CNN
 F 1 "1K" H 6980 4560 50  0000 L CNN
 F 2 "Resistors_ThroughHole:Resistor_Horizontal_RM10mm" H 6950 4600 50  0001 C CNN
@@
 $EndComp
 $Comp
-L R_Small R6
+L R_Small R7
 U 1 1 57205E2D
 P 6950 4800
-F 0 "R6" H 6980 4820 50  0000 L CNN
+F 0 "R7" H 6980 4820 50  0000 L CNN
 F 1 "1K" H 6980 4760 50  0000 L CNN
 F 2 "Resistors_ThroughHole:Resistor_Horizontal_RM10mm" H 6950 4800 50  0001 C CNN
@@
 	7550 4800 7400 4800
 $Comp
-L USB_B CONN1
+L USB_B-RESCUE-DIYduino CONN1
 U 1 1 57207054
 P 1200 5250

Commit message: update
Changed lines of the file:
@@
 LIBS:contrib
 LIBS:valves
-LIBS:LCD7th
 LIBS:DIYduino-cache
 EELAYER 25 0
@@
 	9925 825  9925 475
 Wire Wire Line
-	2450 1200 2450 2300
-Wire Wire Line
 	2450 1800 2550 1800
 Wire Wire Line
@@
 Wire Wire Line
 	2300 2300 2550 2300
-Connection ~ 2450 2300
-Connection ~ 2450 1800
 Wire Wire Line
 	2550 2400 2450 2400
@@
 	1    0    0    -1
 $EndComp
+Wire Wire Line
+	2450 1800 2450 1200
 $EndSCHEMATC
